Commit message: model paths fixed and meshes and config added.

File: urdf/mogi_bot.urdf (robot description, URDF)
Before this commit: robot mogi_bot, 4 links, 3 joints
Links:
- link base_link: geometry collision box size=.4 .2 .1; collision sphere radius=0.0499
- link left_wheel: geometry collision cylinder length=.05 radius=.1; visual mesh filename=package://drone_basic_py/meshes/wheel.dae
- link right_wheel: geometry collision cylinder length=.05 radius=.1; visual mesh filename=package://drone_basic_py/meshes/wheel.dae

File: urdf/mogi_bot_mecanum.urdf (robot description, URDF)
Before this commit: robot mogi_bot, 6 links, 5 joints
Links:
- link base_link: geometry collision box size=.4 .2 .1; visual mesh filename=package://drone_basic_py/meshes/mogi_bot.dae
- link front_left_wheel: geometry collision sphere radius=.1; visual mesh filename=package://drone_basic_py/meshes/mecanum_wheel_left.STL scale=0.002 .002 0.002
- link front_right_wheel: geometry collision sphere radius=.1; visual mesh filename=package://drone_basic_py/meshes/mecanum_wheel_right.STL scale=0.002 .002 0.002
- link rear_left_wheel: geometry collision sphere radius=.1; visual mesh filename=package://drone_basic_py/meshes/mecanum_wheel_right.STL scale=0.002 .002 0.002
- link rear_right_wheel: geometry collision sphere radius=.1; visual mesh filename=package://drone_basic_py/meshes/mecanum_wheel_left.STL scale=0.002 .002 0.002

File: urdf/mogi_bot_skid_steer.urdf (robot description, URDF)
Before this commit: robot mogi_bot, 6 links, 5 joints
Links:
- link base_link: geometry collision box size=.4 .2 .1; visual mesh filename=package://drone_basic_py/meshes/mogi_bot.dae
- link front_left_wheel: geometry collision cylinder length=.05 radius=.1; visual mesh filename=package://drone_basic_py/meshes/wheel.dae
- link front_right_wheel: geometry collision cylinder length=.05 radius=.1; visual mesh filename=package://drone_basic_py/meshes/wheel.dae
- link rear_left_wheel: geometry collision cylinder length=.05 radius=.1; visual mesh filename=package://drone_basic_py/meshes/wheel.dae
- link rear_right_wheel: geometry collision cylinder length=.05 radius=.1; visual mesh filename=package://drone_basic_py/meshes/wheel.dae
