Commit message: check_urdf és spawn drone model

File: urdf/drone_custom.urdf (robot description, URDF)
Before this commit: robot mogi_bot, 2 links, 1 joints
Links:
- link base_link: geometry collision box size=.4 .2 .1; visual mesh filename=package://drone_basic_py/meshes/drone_model_basic.dae

Commit message: Drone model with 4 rotor

File: urdf/drone_custom.urdf (robot description, URDF)
Before this commit: robot drone_custom, 2 links, 1 joints
Links:
- added link rotor_1, mass 0.0001; visual cylinder length=0.02 radius=0.01
- added link rotor_2, mass 0.0001; visual cylinder length=0.02 radius=0.01
- added link rotor_3, mass 0.0001; visual cylinder length=0.02 radius=0.01
- added link rotor_4, mass 0.0001; visual cylinder length=0.02 radius=0.01
- link base_link: mass 15.0 -> 1; geometry collision box size=.1 .4 .4; visual mesh filename=package://drone_basic_py/meshes/drone_model_basic.dae
Joints:
- added joint rotor_1_joint: type fixed, parent base_link, child rotor_1, origin xyz=0.1 0.1 0.0 rpy=0 0 0
- added joint rotor_2_joint: type fixed, parent base_link, child rotor_2, origin xyz=-0.1 0.1 0.0 rpy=0 0 0
- added joint rotor_3_joint: type fixed, parent base_link, child rotor_3, origin xyz=0.1 -0.1 0.0 rpy=0 0 0
- added joint rotor_4_joint: type fixed, parent base_link, child rotor_4, origin xyz=-0.1 -0.1 0.0 rpy=0 0 0

Commit message: Rotor actuators

File: urdf/drone_custom.urdf (robot description, URDF)
Before this commit: robot drone_custom, 6 links, 5 joints
Links:
- link base_link: geometry collision box size=.4 .4 .1; visual mesh filename=package://drone_basic_py/meshes/drone_model_basic.dae

Commit message: First succesful takeoff with direct rotor speed commands

File: urdf/drone_custom.urdf (robot description, URDF)
Before this commit: robot drone_custom, 6 links, 5 joints
Links:
- removed link base_footprint
- removed link base_link
- removed link rotor_1
- removed link rotor_2
- removed link rotor_3
- removed link rotor_4
- added link drone/base_footprint
- added link drone/base_link, mass 1; collision box size=.4 .4 .1; visual mesh filename=package://drone_basic_py/meshes/drone_model_basic.dae
- added link drone/rotor_0, mass 0.005; collision cylinder length=0.005 radius=0.1; visual mesh filename=package://drone_basic_py/meshes/propeller_ccw.dae scale=0.08 0.08 0.08
- added link drone/rotor_1, mass 0.005; collision cylinder length=0.005 radius=0.1; visual mesh filename=package://drone_basic_py/meshes/propeller_ccw.dae scale=0.08 0.08 0.08
- added link drone/rotor_2, mass 0.005; collision cylinder length=0.005 radius=0.1; visual mesh filename=package://drone_basic_py/meshes/propeller_cw.dae scale=0.08 0.08 0.08
- added link drone/rotor_3, mass 0.005; collision cylinder length=0.005 radius=0.1; visual mesh filename=package://drone_basic_py/meshes/propeller_cw.dae scale=0.08 0.08 0.08
Joints:
- removed joint base_footprint_joint
- removed joint rotor_1_joint
- removed joint rotor_2_joint
- removed joint rotor_3_joint
- removed joint rotor_4_joint
- added joint drone/base_footprint_joint: type fixed, parent drone/base_footprint, child drone/base_link, origin xyz=0 0 0 rpy=0 0 0
- added joint drone/rotor_0_joint: type continuous, parent drone/base_link, child drone/rotor_0, origin xyz=0.1 -0.1 0.023 rpy=0 0 0, axis 0 0 1
- added joint drone/rotor_1_joint: type continuous, parent drone/base_link, child drone/rotor_1, origin xyz=-0.1 0.1 0.023 rpy=0 0 0, axis 0 0 1
- added joint drone/rotor_2_joint: type continuous, parent drone/base_link, child drone/rotor_2, origin xyz=0.1 0.1 0.023 rpy=0 0 0, axis 0 0 1
- added joint drone/rotor_3_joint: type continuous, parent drone/base_link, child drone/rotor_3, origin xyz=-0.1 -0.1 0.023 rpy=0 0 0, axis 0 0 1

Commit message: camera added onto the drone, Working at 3hz.

File: urdf/drone_custom.urdf (robot description, URDF)
Before this commit: robot drone, 6 links, 5 joints
Links:
- added link camera_link, mass 0.0; collision box size=.03 .03 .03; visual box size=.03 .03 .03
- added link camera_link_optical
Joints:
- added joint camera_joint: type fixed, parent drone/base_link, child camera_link, origin xyz=0.2 0 0.0 rpy=0 0 0, axis 0 1 0
- added joint camera_optical_joint: type fixed, parent camera_link, child camera_link_optical, origin xyz=0 0 0 rpy=-1.5707 0 -1.5707

Commit message: imu added, camera image shaking fixed

File: urdf/drone_custom.urdf (robot description, URDF)
Before this commit: robot drone, 8 links, 7 joints
Links:
- added link imu_link
Joints:
- added joint imu_joint: type fixed, parent drone/base_link, child imu_link, origin xyz=0 0 0 rpy=0 0 0

Commit message: First working state estimation with EKF and navsat transformer

File: urdf/drone_custom.urdf (robot description, URDF)
Before this commit: robot drone, 9 links, 8 joints
Links:
- added link navsat_link
Joints:
- added joint navsat_joint: type fixed, parent drone/base_link, child navsat_link, origin xyz=0 0 0 rpy=0 0 0

Commit message: New Drone modell

File: urdf/drone_custom.urdf (robot description, URDF)
Before this commit: robot drone, 10 links, 9 joints
Links:
- link camera_link: geometry collision cylinder length=0.03 radius=0.015; visual cylinder length=0.03 radius=0.03
- link drone/base_link: geometry collision box size=.4 .4 .102; visual mesh filename=package://drone_basic_py/meshes/drone_model_v2.dae
Joints:
- joint camera_joint: origin xyz=0.2 0 0.0 rpy=0 0 0 -> xyz=0.18 0 -0.02 rpy=0 0 0
